File: attache rev k.kicad_pcb (KiCad board)
At the start: 2 copper layers, 373 x 126 mm, 247 parts, among them J1 USB_mini_micro_B, K0 KEYSW, K1 KEYSW, K10 KEYSW, K100 KEYSW, K101 KEYSW, K102 KEYSW, K103 KEYSW, K104 KEYSW, K105 KEYSW, K106 KEYSW, K107 KEYSW, K108 KEYSW, K109 KEYSW, K11 KEYSW, K110 KEYSW, K12 KEYSW, K13 KEYSW, K14 KEYSW, K15 KEYSW, K16 KEYSW, K17 KEYSW, K18 KEYSW, K19 KEYSW, K2 KEYSW, K20 KEYSW, K21 KEYSW, K22 KEYSW, K23 KEYSW, K24 KEYSW, K25 KEYSW, K26 KEYSW, K27 KEYSW, K28 KEYSW, K29 KEYSW, K3 KEYSW, K30 KEYSW, K31 KEYSW, K32 KEYSW, K33 KEYSW, K34 KEYSW, K35 KEYSW, K36 KEYSW, K37 KEYSW, K38 KEYSW, K39 KEYSW, K4 KEYSW, K40 KEYSW, K41 KEYSW, K42 KEYSW, K43 KEYSW, K44 KEYSW, K45 KEYSW, K46 KEYSW, K47 KEYSW, K48 KEYSW, K49 KEYSW, K5 KEYSW, K50 KEYSW, K51 KEYSW, K52 KEYSW, K53 KEYSW, K54 KEYSW, K55 KEYSW, K56 KEYSW, K57 KEYSW, K58 KEYSW, K59 KEYSW, K6 KEYSW, K60 KEYSW, K61 KEYSW, K62 KEYSW, K63 KEYSW, K64 KEYSW, K65 KEYSW, K66 KEYSW, K67 KEYSW, K68 KEYSW, K69 KEYSW, K7 KEYSW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

Commit message: Attache
Parts:
- added K111: KEYSW, cherry:SW_PCB_2PIN, F.Cu at (35.7, 126.2)
- added K112: KEYSW, cherry:SW_PCB_2PIN, F.Cu at (57.1, 126.2)
- moved D4 16.4 mm to (42.5, 116.2), turned to 0 degrees
Routing:
- net row4: track 465.3 -> 486.6 mm
- net col1: track 402.8 -> 420.1 mm
- net Net-(D9-Pad2): track 7.47 -> 13.0 mm
- net col0: track 414.1 -> 419.0 mm
- net Net-(D4-Pad2): track 21.2 -> 23.3 mm
Other:
- board text added: "1.25u Shift"
- board text added: "1u Any"
