File: attache rev k.sch (KiCad schematic (older format))
At the start: 226 parts, among them J1 USB_mini_micro_B, K0 KEYSW, K1 KEYSW, K10 KEYSW, K100 KEYSW, K101 KEYSW, K102 KEYSW, K103 KEYSW, K104 KEYSW, K105 KEYSW, K106 KEYSW, K107 KEYSW, K108 KEYSW, K109 KEYSW, K11 KEYSW, K110 KEYSW, K12 KEYSW, K13 KEYSW, K14 KEYSW, K15 KEYSW, K16 KEYSW, K17 KEYSW, K18 KEYSW, K19 KEYSW, K2 KEYSW, K20 KEYSW, K21 KEYSW, K22 KEYSW, K23 KEYSW, K24 KEYSW, K25 KEYSW, K26 KEYSW, K27 KEYSW, K28 KEYSW, K29 KEYSW, K3 KEYSW, K30 KEYSW, K31 KEYSW, K32 KEYSW, K33 KEYSW, K34 KEYSW, K35 KEYSW, K36 KEYSW, K37 KEYSW, K38 KEYSW, K39 KEYSW, K4 KEYSW, K40 KEYSW, K41 KEYSW, K42 KEYSW, K43 KEYSW, K44 KEYSW, K45 KEYSW, K46 KEYSW, K47 KEYSW, K48 KEYSW, K49 KEYSW, K5 KEYSW, K50 KEYSW, K51 KEYSW, K52 KEYSW, K53 KEYSW, K54 KEYSW, K55 KEYSW, K56 KEYSW, K57 KEYSW, K58 KEYSW, K59 KEYSW, K6 KEYSW, K60 KEYSW, K61 KEYSW, K62 KEYSW, K63 KEYSW, K64 KEYSW, K65 KEYSW, K66 KEYSW, K67 KEYSW, K68 KEYSW, K69 KEYSW, K7 KEYSW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

Commit message: Attache
Parts:
- added K111, K112: KEYSW, cherry:SW_PCB_2PIN, symbol KEYSW
Connections:
- net col0: now also K111.2
- net col1: now also K112.2
- net at D4.2, K102.1, K4.1: now also K111.1
- net at D9.2, K9.1: now also K112.1
Other:
- moved on the sheet: D9
Changed lines of the file:
@@
 L D D9
 U 1 1 5911A364
-P 4500 5350
-F 0 "D9" H 4350 5300 60  0000 C CNN
-F 1 "D" V 4650 5300 60  0001 C CNN
-F 2 "keyboard_parts:D_SOD123_axial" H 4500 5350 60  0001 C CNN
-F 3 "" H 4500 5350 60  0000 C CNN
-	1    4500 5350
+P 4600 5350
+F 0 "D9" H 4450 5300 60  0000 C CNN
+F 1 "D" V 4750 5300 60  0001 C CNN
+F 2 "keyboard_parts:D_SOD123_axial" H 4600 5350 60  0001 C CNN
+F 3 "" H 4600 5350 60  0000 C CNN
+	1    4600 5350
 	-1   0    0    1
 $EndComp
@@
 Connection ~ 4500 5450
 Wire Wire Line
-	4500 5200 4500 5150
+	4500 5150 4500 5300
 Wire Wire Line
 	4500 5000 4500 4950
@@
 Connection ~ 11100 5600
 Connection ~ 11900 5600
-Wire Wire Line
-	3100 2250 3100 5700
 Connection ~ 3700 5650
 Wire Wire Line
@@
 Connection ~ 3900 2500
 NoConn ~ 9400 9300
+$Comp
+L KEYSW K112
+U 1 1 59928C28
+P 4200 5300
+F 0 "K112" H 4150 5300 60  0000 C CNN
+F 1 "KEYSW" H 4200 5200 60  0001 C CNN
+F 2 "cherry:SW_PCB_2PIN" H 4200 5300 60  0001 C CNN
+F 3 "" H 4200 5300 60  0000 C CNN
+	1    4200 5300
+	1    0    0    -1
+$EndComp
+$Comp
+L KEYSW K111
+U 1 1 599290BF
+P 3400 5400
+F 0 "K111" H 3350 5400 60  0000 C CNN
+F 1 "KEYSW" H 3400 5300 60  0001 C CNN
+F 2 "cherry:SW_PCB_2PIN" H 3400 5400 60  0001 C CNN
+F 3 "" H 3400 5400 60  0000 C CNN
+	1    3400 5400
+	1    0    0    -1
+$EndComp
+Wire Wire Line
+	3100 2250 3100 5700
+Connection ~ 3900 5300
+Wire Wire Line
+	4500 5200 4600 5200
+Connection ~ 4500 5200
+Wire Wire Line
+	4500 5400 4600 5400
+Connection ~ 3100 5400
+Wire Wire Line
+	3700 5400 3700 5350
+Wire Wire Line
+	3700 5350 3750 5350
+Wire Wire Line
+	3750 5350 3750 5200
+Connection ~ 3750 5200
 $EndSCHEMATC
